Commit message: urdf update

File: scara_description/urdf/arm.xacro (robot description, xacro)
@@ -34,5 +34,5 @@
         <child link="column_link"/>
         <axis xyz="0 0 1"/>
-        <limit lower="-1.57" upper="1.57" effort="10.0" velocity="1.5" />
+        <limit lower="-2.0" upper="2.0" effort="10.0" velocity="1.5" />
     </joint>
     <link name="shoulder_link">
@@ -48,13 +48,13 @@
     </link>
     <joint name="shoulder_joint" type="prismatic">
-        <origin xyz="0.0 0.0 0.3" rpy="0.0 0.0 0.0"/>
+        <origin xyz="0.0 0.0 0.28" rpy="0.0 0.0 0.0"/>
         <parent link="column_link"/>
         <child link="shoulder_link"/>
         <axis xyz="0 0 1"/>
-        <limit effort="100.0" velocity="0.5" lower="0.0" upper="-0.15"/>
+        <limit effort="100.0" velocity="0.5" lower="0.0" upper="-0.21"/>
     </joint>
     <link name="forearm_link">
         <visual>
-            <origin xyz="-0.0 0.0 -0.0" rpy="0.0 0.0 0.0"/>
+            <origin xyz="-0.273 0.0 -0.351" rpy="0.0 0.0 0.0"/>
             <geometry>
                 <mesh filename="package://scara_description/meshes/forearm_link.stl" scale="0.001 0.001 0.001"/>
@@ -65,10 +65,10 @@
         </visual>
     </link>
-    <joint name="shoulder_joint" type="prismatic">
-        <origin xyz="0.0 0.0 0.0" rpy="0.0 0.0 0.0"/>
-        <parent link="column_link"/>
-        <child link="shoulder_link"/>
+    <joint name="forearm_joint" type="revolute">
+        <origin xyz="0.228 0.0 -0.04" rpy="0.0 0.0 0.0"/>
+        <parent link="shoulder_link"/>
+        <child link="forearm_link"/>
         <axis xyz="0 0 1"/>
-        <limit lower="-1.57" upper="1.57" effort="10.0" velocity="1.5" />
+        <limit lower="-2.0" upper="2.0" effort="10.0" velocity="1.5" />
     </joint>
 </robot>

Commit message: urdf wrist update

File: scara_description/urdf/arm.xacro (robot description, xacro)
@@ -72,3 +72,21 @@
         <limit lower="-2.0" upper="2.0" effort="10.0" velocity="1.5" />
     </joint>
+    <link name="wrist_link">
+        <visual>
+            <origin xyz="-0.4095 0.0 -0.291" rpy="0.0 0.0 0.0"/>
+            <geometry>
+                <mesh filename="package://scara_description/meshes/wrist_link.stl" scale="0.001 0.001 0.001"/>
+            </geometry>
+            <material name="grey">
+                <color rgba="0.8 0.8 0.8 1.0"/>
+            </material>
+        </visual>
+    </link>
+    <joint name="wrist_joint" type="revolute">
+        <origin xyz="0.1365 0.0 -0.06" rpy="0.0 0.0 0.0"/>
+        <parent link="forearm_link"/>
+        <child link="wrist_link"/>
+        <axis xyz="0 0 1"/>
+        <limit lower="-2.0" upper="2.0" effort="10.0" velocity="1.5" />
+    </joint>
 </robot>

Commit message: full urdf scara

File: scara_description/urdf/arm.xacro (robot description, xacro)
@@ -52,5 +52,5 @@
         <child link="shoulder_link"/>
         <axis xyz="0 0 1"/>
-        <limit effort="100.0" velocity="0.5" lower="0.0" upper="-0.21"/>
+        <limit effort="100.0" velocity="0.5" lower="0.0" upper="-0.15"/>
     </joint>
     <link name="forearm_link">
@@ -90,3 +90,39 @@
         <limit lower="-2.0" upper="2.0" effort="10.0" velocity="1.5" />
     </joint>
+    <link name="left_finger_link">
+        <visual>
+            <origin xyz="-0.409 -0.0626 -0.2775" rpy="0.0 0.0 0.0"/>
+            <geometry>
+                <mesh filename="package://scara_description/meshes/left_finger_link.stl" scale="0.001 0.001 0.001"/>
+            </geometry>
+            <material name="grey">
+                <color rgba="0.8 0.8 0.8 1.0"/>
+            </material>
+        </visual>
+    </link>
+    <joint name="left_finger_joint" type="prismatic">
+        <origin xyz="0.0 0.064 -0.0135" rpy="0.0 0.0 0.0"/>
+        <parent link="wrist_link"/>
+        <child link="left_finger_link"/>
+        <axis xyz="0 1 0"/>
+        <limit effort="100.0" velocity="0.5" lower="0.0" upper="-0.02"/>
+    </joint>
+    <link name="right_finger_link">
+        <visual>
+            <origin xyz="-0.409 0.0626 -0.2775" rpy="0.0 0.0 0.0"/>
+            <geometry>
+                <mesh filename="package://scara_description/meshes/right_finger_link.stl" scale="0.001 0.001 0.001"/>
+            </geometry>
+            <material name="grey">
+                <color rgba="0.8 0.8 0.8 1.0"/>
+            </material>
+        </visual>
+    </link>
+    <joint name="right_finger_joint" type="prismatic">
+        <origin xyz="0.0 -0.064 -0.0135" rpy="0.0 0.0 0.0"/>
+        <parent link="wrist_link"/>
+        <child link="right_finger_link"/>
+        <axis xyz="0 -1 0"/>
+        <limit effort="100.0" velocity="0.5" lower="0.0" upper="-0.02"/>
+    </joint>
 </robot>

Commit message: gazebo spawn added

File: scara_description/urdf/arm.xacro (robot description, xacro)
@@ -4,15 +4,30 @@
     <link name="base_link">
         <visual>
-            <origin xyz="0.0 0.0 0.0" rpy="0.0 0.0 0.0"/>
-            <geometry>
-                <mesh filename="package://scara_description/meshes/base_link.stl" scale="0.001 0.001 0.001"/>
-            </geometry>
-            <material name="grey">
-                <color rgba="0.8 0.8 0.8 1.0"/>
-            </material>
-        </visual>
+            <origin xyz="0 0 0" rpy="0 0 0"/>
+            <geometry>
+                <mesh filename="package://scara_description/meshes/base_link.stl"
+                      scale="0.001 0.001 0.001"/>
+            </geometry>
+            <material name="grey">
+                <color rgba="0.8 0.8 0.8 1.0"/>
+            </material>
+        </visual>
+        <collision>
+            <origin xyz="0 0 0" rpy="0 0 0"/>
+            <geometry>
+                <mesh filename="package://scara_description/meshes/base_link.stl"
+                      scale="0.001 0.001 0.001"/>
+            </geometry>
+        </collision>
+        <inertial>
+            <origin xyz="0 0 0" rpy="0 0 0"/>
+            <mass value="5.0"/>
+            <inertia ixx="0.01" ixy="0.0" ixz="0.0"
+                               iyy="0.01" iyz="0.0"
+                               izz="0.01"/>
+        </inertial>
     </link>
     <joint name="base_joint" type="fixed">
-        <origin xyz="0.0 0.0 0.0" rpy="0.0 0.0 0.0"/>
+        <origin xyz="0 0 0" rpy="0 0 0"/>
         <parent link="world"/>
         <child link="base_link"/>
@@ -20,109 +35,214 @@
     <link name="column_link">
         <visual>
-            <origin xyz="-0.045 0.0 -0.089" rpy="0.0 0.0 0.0"/>
-            <geometry>
-                <mesh filename="package://scara_description/meshes/column_link.stl" scale="0.001 0.001 0.001"/>
-            </geometry>
-            <material name="grey">
-                <color rgba="0.8 0.8 0.8 1.0"/>
-            </material>
-        </visual>
+            <origin xyz="-0.045 0 -0.089" rpy="0 0 0"/>
+            <geometry>
+                <mesh filename="package://scara_description/meshes/column_link.stl"
+                      scale="0.001 0.001 0.001"/>
+            </geometry>
+            <material name="grey">
+                <color rgba="0.8 0.8 0.8 1.0"/>
+            </material>
+        </visual>
+        <collision>
+            <origin xyz="-0.045 0 -0.089" rpy="0 0 0"/>
+            <geometry>
+                <mesh filename="package://scara_description/meshes/column_link.stl"
+                      scale="0.001 0.001 0.001"/>
+            </geometry>
+        </collision>
+        <inertial>
+            <origin xyz="-0.045 0 -0.089" rpy="0 0 0"/>
+            <mass value="4.0"/>
+            <inertia ixx="0.01" ixy="0.0" ixz="0.0"
+                               iyy="0.01" iyz="0.0"
+                               izz="0.01"/>
+        </inertial>
     </link>
     <joint name="column_joint" type="revolute">
-        <origin xyz="0.045 0.0 0.089" rpy="0.0 0.0 0.0"/>
+        <origin xyz="0.045 0 0.089" rpy="0 0 0"/>
         <parent link="base_link"/>
         <child link="column_link"/>
         <axis xyz="0 0 1"/>
-        <limit lower="-2.0" upper="2.0" effort="10.0" velocity="1.5" />
+        <limit lower="-2.0" upper="2.0" effort="10.0" velocity="1.5"/>
     </joint>
     <link name="shoulder_link">
         <visual>
-            <origin xyz="-0.045 0.0 -0.39" rpy="0.0 0.0 0.0"/>
-            <geometry>
-                <mesh filename="package://scara_description/meshes/shoulder_link.stl" scale="0.001 0.001 0.001"/>
-            </geometry>
-            <material name="grey">
-                <color rgba="0.8 0.8 0.8 1.0"/>
-            </material>
-        </visual>
+            <origin xyz="-0.045 0 -0.39" rpy="0 0 0"/>
+            <geometry>
+                <mesh filename="package://scara_description/meshes/shoulder_link.stl"
+                      scale="0.001 0.001 0.001"/>
+            </geometry>
+            <material name="grey">
+                <color rgba="0.8 0.8 0.8 1.0"/>
+            </material>
+        </visual>
+        <collision>
+            <origin xyz="-0.045 0 -0.39" rpy="0 0 0"/>
+            <geometry>
+                <mesh filename="package://scara_description/meshes/shoulder_link.stl"
+                      scale="0.001 0.001 0.001"/>
+            </geometry>
+        </collision>
+        <inertial>
+            <origin xyz="-0.045 0 -0.39" rpy="0 0 0"/>
+            <mass value="3.0"/>
+            <inertia ixx="0.01" ixy="0.0" ixz="0.0"
+                               iyy="0.01" iyz="0.0"
+                               izz="0.01"/>
+        </inertial>
     </link>
     <joint name="shoulder_joint" type="prismatic">
-        <origin xyz="0.0 0.0 0.28" rpy="0.0 0.0 0.0"/>
+        <origin xyz="0 0 0.28" rpy="0 0 0"/>
         <parent link="column_link"/>
         <child link="shoulder_link"/>
         <axis xyz="0 0 1"/>
-        <limit effort="100.0" velocity="0.5" lower="0.0" upper="-0.15"/>
+        <limit lower="-0.15" upper="0.0"
+               effort="100.0"
+               velocity="0.5"/>
     </joint>
     <link name="forearm_link">
         <visual>
-            <origin xyz="-0.273 0.0 -0.351" rpy="0.0 0.0 0.0"/>
-            <geometry>
-                <mesh filename="package://scara_description/meshes/forearm_link.stl" scale="0.001 0.001 0.001"/>
-            </geometry>
-            <material name="grey">
-                <color rgba="0.8 0.8 0.8 1.0"/>
-            </material>
-        </visual>
+            <origin xyz="-0.273 0 -0.351" rpy="0 0 0"/>
+            <geometry>
+                <mesh filename="package://scara_description/meshes/forearm_link.stl"
+                      scale="0.001 0.001 0.001"/>
+            </geometry>
+            <material name="grey">
+                <color rgba="0.8 0.8 0.8 1.0"/>
+            </material>
+        </visual>
+        <collision>
+            <origin xyz="-0.273 0 -0.351" rpy="0 0 0"/>
+            <geometry>
+                <mesh filename="package://scara_description/meshes/forearm_link.stl"
+                      scale="0.001 0.001 0.001"/>
+            </geometry>
+        </collision>
+        <inertial>
+            <origin xyz="-0.273 0 -0.351" rpy="0 0 0"/>
+            <mass value="2.0"/>
+            <inertia ixx="0.01" ixy="0.0" ixz="0.0"
+                               iyy="0.01" iyz="0.0"
+                               izz="0.01"/>
+        </inertial>
     </link>
     <joint name="forearm_joint" type="revolute">
-        <origin xyz="0.228 0.0 -0.04" rpy="0.0 0.0 0.0"/>
+        <origin xyz="0.228 0 -0.04" rpy="0 0 0"/>
         <parent link="shoulder_link"/>
         <child link="forearm_link"/>
         <axis xyz="0 0 1"/>
-        <limit lower="-2.0" upper="2.0" effort="10.0" velocity="1.5" />
+        <limit lower="-2.0" upper="2.0"
+               effort="10.0"
+               velocity="1.5"/>
     </joint>
     <link name="wrist_link">
         <visual>
-            <origin xyz="-0.4095 0.0 -0.291" rpy="0.0 0.0 0.0"/>
-            <geometry>
-                <mesh filename="package://scara_description/meshes/wrist_link.stl" scale="0.001 0.001 0.001"/>
-            </geometry>
-            <material name="grey">
-                <color rgba="0.8 0.8 0.8 1.0"/>
-            </material>
-        </visual>
+            <origin xyz="-0.4095 0 -0.291" rpy="0 0 0"/>
+            <geometry>
+                <mesh filename="package://scara_description/meshes/wrist_link.stl"
+                      scale="0.001 0.001 0.001"/>
+            </geometry>
+            <material name="grey">
+                <color rgba="0.8 0.8 0.8 1.0"/>
+            </material>
+        </visual>
+        <collision>
+            <origin xyz="-0.4095 0 -0.291" rpy="0 0 0"/>
+            <geometry>
+                <mesh filename="package://scara_description/meshes/wrist_link.stl"
+                      scale="0.001 0.001 0.001"/>
+            </geometry>
+        </collision>
+        <inertial>
+            <origin xyz="-0.4095 0 -0.291" rpy="0 0 0"/>
+            <mass value="1.5"/>
+            <inertia ixx="0.01" ixy="0.0" ixz="0.0"
+                               iyy="0.01" iyz="0.0"
+                               izz="0.01"/>
+        </inertial>
     </link>
     <joint name="wrist_joint" type="revolute">
-        <origin xyz="0.1365 0.0 -0.06" rpy="0.0 0.0 0.0"/>
+        <origin xyz="0.1365 0 -0.06" rpy="0 0 0"/>
         <parent link="forearm_link"/>
         <child link="wrist_link"/>
         <axis xyz="0 0 1"/>
-        <limit lower="-2.0" upper="2.0" effort="10.0" velocity="1.5" />
+        <limit lower="-2.0" upper="2.0"
+               effort="10.0"
+               velocity="1.5"/>
     </joint>
     <link name="left_finger_link">
         <visual>
-            <origin xyz="-0.409 -0.0626 -0.2775" rpy="0.0 0.0 0.0"/>
-            <geometry>
-                <mesh filename="package://scara_description/meshes/left_finger_link.stl" scale="0.001 0.001 0.001"/>
-            </geometry>
-            <material name="grey">
-                <color rgba="0.8 0.8 0.8 1.0"/>
-            </material>
-        </visual>
-    </link>
+            <origin xyz="-0.409 -0.0626 -0.2775" rpy="0 0 0"/>
+            <geometry>
+                <mesh filename="package://scara_description/meshes/left_finger_link.stl"
+                      scale="0.001 0.001 0.001"/>
+            </geometry>
+            <material name="grey">
+                <color rgba="0.8 0.8 0.8 1.0"/>
+            </material>
+        </visual>
+        <collision>
+            <origin xyz="-0.409 -0.0626 -0.2775" rpy="0 0 0"/>
+            <geometry>
+                <mesh filename="package://scara_description/meshes/left_finger_link.stl"
+                      scale="0.001 0.001 0.001"/>
+            </geometry>
+        </collision>
+        <inertial>
+            <origin xyz="-0.409 -0.0626 -0.2775" rpy="0 0 0"/>
+            <mass value="1.0"/>
+            <inertia ixx="0.01" ixy="0.0" ixz="0.0"
+                               iyy="0.01" iyz="0.0"
+                               izz="0.01"/>
+        </inertial>
+    </link>
+    <!-- MASTER GRIPPER JOINT -->
     <joint name="left_finger_joint" type="prismatic">
-        <origin xyz="0.0 0.064 -0.0135" rpy="0.0 0.0 0.0"/>
+        <origin xyz="0 0.064 -0.0135" rpy="0 0 0"/>
         <parent link="wrist_link"/>
         <child link="left_finger_link"/>
         <axis xyz="0 1 0"/>
-        <limit effort="100.0" velocity="0.5" lower="0.0" upper="-0.02"/>
+        <limit lower="-0.02" upper="0.0"
+               effort="100.0"
+               velocity="0.5"/>
     </joint>
     <link name="right_finger_link">
         <visual>
-            <origin xyz="-0.409 0.0626 -0.2775" rpy="0.0 0.0 0.0"/>
-            <geometry>
-                <mesh filename="package://scara_description/meshes/right_finger_link.stl" scale="0.001 0.001 0.001"/>
-            </geometry>
-            <material name="grey">
-                <color rgba="0.8 0.8 0.8 1.0"/>
-            </material>
-        </visual>
-    </link>
+            <origin xyz="-0.409 0.0626 -0.2775" rpy="0 0 0"/>
+            <geometry>
+                <mesh filename="package://scara_description/meshes/right_finger_link.stl"
+                      scale="0.001 0.001 0.001"/>
+            </geometry>
+            <material name="grey">
+                <color rgba="0.8 0.8 0.8 1.0"/>
+            </material>
+        </visual>
+        <collision>
+            <origin xyz="-0.409 0.0626 -0.2775" rpy="0 0 0"/>
+            <geometry>
+                <mesh filename="package://scara_description/meshes/right_finger_link.stl"
+                      scale="0.001 0.001 0.001"/>
+            </geometry>
+        </collision>
+        <inertial>
+            <origin xyz="-0.409 0.0626 -0.2775" rpy="0 0 0"/>
+            <mass value="1.0"/>
+            <inertia ixx="0.01" ixy="0.0" ixz="0.0"
+                               iyy="0.01" iyz="0.0"
+                               izz="0.01"/>
+        </inertial>
+    </link>
+    <!-- MIMIC JOINT -->
     <joint name="right_finger_joint" type="prismatic">
-        <origin xyz="0.0 -0.064 -0.0135" rpy="0.0 0.0 0.0"/>
+        <origin xyz="0 -0.064 -0.0135" rpy="0 0 0"/>
         <parent link="wrist_link"/>
         <child link="right_finger_link"/>
         <axis xyz="0 -1 0"/>
-        <limit effort="100.0" velocity="0.5" lower="0.0" upper="-0.02"/>
+        <limit lower="-0.02" upper="0.0"
+               effort="100.0"
+               velocity="0.5"/>
+        <mimic joint="left_finger_joint"
+               multiplier="1.0"
+               offset="0.0"/>
     </joint>
 </robot>

File: scara_description/urdf/scara.urdf.xacro (robot description, xacro)
@@ -4,3 +4,5 @@
     <xacro:arg name="is_sim" default="true"/>
     <xacro:include filename="$(find scara_description)/urdf/arm.xacro" />
+    <xacro:include filename="$(find scara_description)/urdf/gazebo.xacro" />
+    <xacro:include filename="$(find scara_description)/urdf/ros2control.xacro" />
 </robot>

Commit message: final working teleop

File: scara_description/urdf/arm.xacro (robot description, xacro)
@@ -97,5 +97,5 @@
         <child link="shoulder_link"/>
         <axis xyz="0 0 1"/>
-        <limit lower="-0.15" upper="0.0"
+        <limit lower="-0.12" upper="0.02"
                effort="100.0"
                velocity="0.5"/>

File: scara_description/urdf/ros2control.xacro (robot description, xacro)
@@ -2,11 +2,10 @@
 <robot xmlns:xacro="http://www.ros.org/wiki/xacro" name="scara">
     <xacro:property name="PI" value="3.14159265359"/>
-    <xacro:arg name="is_sim"       default="true"/>
-    <xacro:arg name="is_ignition"  default="false"/>
+    <xacro:arg name="is_sim"      default="true"/>
+    <xacro:arg name="is_ignition" default="false"/>
     <ros2_control name="RobotSystem" type="system">
-        <!-- ── No Gazebo: slider GUI / standalone testing ── -->
         <xacro:if value="$(arg is_sim)">
             <xacro:if value="$(arg is_ignition)">
-                <!-- ROS 2 Humble + Ignition Fortress -->
+                <!-- Ignition Fortress (ROS 2 Humble) -->
                 <hardware>
                     <plugin>ign_ros2_control/IgnitionSystem</plugin>
@@ -14,5 +13,5 @@
             </xacro:if>
             <xacro:unless value="$(arg is_ignition)">
-                <!-- ROS 2 Iron+ + Gazebo Garden/Harmonic -->
+                <!-- Gazebo Garden/Harmonic (ROS 2 Iron+) -->
                 <hardware>
                     <plugin>gz_ros2_control/GazeboSimSystem</plugin>
@@ -20,5 +19,5 @@
             </xacro:unless>
         </xacro:if>
-        <!-- ── No Gazebo: slider GUI / standalone testing ── -->
+        <!-- Standalone / slider GUI — no Gazebo -->
         <xacro:unless value="$(arg is_sim)">
             <hardware>
@@ -62,5 +61,5 @@
             <state_interface name="velocity"/>
         </joint>
-        <!-- Master Gripper Joint -->
+        <!-- Master Gripper — command interface here -->
         <joint name="left_finger_joint">
             <command_interface name="position">
@@ -71,5 +70,5 @@
             <state_interface name="velocity"/>
         </joint>
-        <!-- Mimic Joint (no command interface) -->
+        <!-- Mimic Joint — state only, no command interface -->
         <joint name="right_finger_joint">
             <param name="mimic">left_finger_joint</param>
