Commit message: materials added

File: scara_description/urdf/arm.xacro (robot description, xacro)
@@ -2,4 +2,5 @@
 <robot name="scara" xmlns:xacro="http://www.ros.org/wiki/xacro">
     <link name="world"/>
+    <!-- ── BASE ─────────────────────────────────────── -->
     <link name="base_link">
         <visual>
@@ -9,7 +10,5 @@
                       scale="0.001 0.001 0.001"/>
             </geometry>
-            <material name="grey">
-                <color rgba="0.8 0.8 0.8 1.0"/>
-            </material>
+            <material name="scara_mid_blue"/>
         </visual>
         <collision>
@@ -33,4 +32,5 @@
         <child link="base_link"/>
     </joint>
+    <!-- ── COLUMN ────────────────────────────────────── -->
     <link name="column_link">
         <visual>
@@ -40,7 +40,5 @@
                       scale="0.001 0.001 0.001"/>
             </geometry>
-            <material name="grey">
-                <color rgba="0.8 0.8 0.8 1.0"/>
-            </material>
+            <material name="scara_mid_blue"/>
         </visual>
         <collision>
@@ -66,4 +64,5 @@
         <limit lower="-2.0" upper="2.0" effort="10.0" velocity="1.5"/>
     </joint>
+    <!-- ── SHOULDER ──────────────────────────────────── -->
     <link name="shoulder_link">
         <visual>
@@ -73,7 +72,5 @@
                       scale="0.001 0.001 0.001"/>
             </geometry>
-            <material name="grey">
-                <color rgba="0.8 0.8 0.8 1.0"/>
-            </material>
+            <material name="scara_mid_blue"/>
         </visual>
         <collision>
@@ -97,8 +94,7 @@
         <child link="shoulder_link"/>
         <axis xyz="0 0 1"/>
-        <limit lower="-0.12" upper="0.02"
-               effort="100.0"
-               velocity="0.5"/>
-    </joint>
+        <limit lower="-0.12" upper="0.02" effort="100.0" velocity="0.5"/>
+    </joint>
+    <!-- ── FOREARM ───────────────────────────────────── -->
     <link name="forearm_link">
         <visual>
@@ -108,7 +104,5 @@
                       scale="0.001 0.001 0.001"/>
             </geometry>
-            <material name="grey">
-                <color rgba="0.8 0.8 0.8 1.0"/>
-            </material>
+            <material name="scara_mid_blue"/>
         </visual>
         <collision>
@@ -132,8 +126,7 @@
         <child link="forearm_link"/>
         <axis xyz="0 0 1"/>
-        <limit lower="-2.0" upper="2.0"
-               effort="10.0"
-               velocity="1.5"/>
-    </joint>
+        <limit lower="-2.0" upper="2.0" effort="10.0" velocity="1.5"/>
+    </joint>
+    <!-- ── WRIST ─────────────────────────────────────── -->
     <link name="wrist_link">
         <visual>
@@ -143,7 +136,5 @@
                       scale="0.001 0.001 0.001"/>
             </geometry>
-            <material name="grey">
-                <color rgba="0.8 0.8 0.8 1.0"/>
-            </material>
+            <material name="scara_dark_blue"/>
         </visual>
         <collision>
@@ -167,8 +158,7 @@
         <child link="wrist_link"/>
         <axis xyz="0 0 1"/>
-        <limit lower="-2.0" upper="2.0"
-               effort="10.0"
-               velocity="1.5"/>
-    </joint>
+        <limit lower="-2.0" upper="2.0" effort="10.0" velocity="1.5"/>
+    </joint>
+    <!-- ── LEFT FINGER ───────────────────────────────── -->
     <link name="left_finger_link">
         <visual>
@@ -178,7 +168,5 @@
                       scale="0.001 0.001 0.001"/>
             </geometry>
-            <material name="grey">
-                <color rgba="0.8 0.8 0.8 1.0"/>
-            </material>
+            <material name="scara_light_grey"/>
         </visual>
         <collision>
@@ -203,8 +191,7 @@
         <child link="left_finger_link"/>
         <axis xyz="0 1 0"/>
-        <limit lower="-0.02" upper="0.0"
-               effort="100.0"
-               velocity="0.5"/>
-    </joint>
+        <limit lower="-0.02" upper="0.0" effort="100.0" velocity="0.5"/>
+    </joint>
+    <!-- ── RIGHT FINGER ──────────────────────────────── -->
     <link name="right_finger_link">
         <visual>
@@ -214,7 +201,5 @@
                       scale="0.001 0.001 0.001"/>
             </geometry>
-            <material name="grey">
-                <color rgba="0.8 0.8 0.8 1.0"/>
-            </material>
+            <material name="scara_light_grey"/>
         </visual>
         <collision>
@@ -239,10 +224,6 @@
         <child link="right_finger_link"/>
         <axis xyz="0 -1 0"/>
-        <limit lower="-0.02" upper="0.0"
-               effort="100.0"
-               velocity="0.5"/>
-        <mimic joint="left_finger_joint"
-               multiplier="1.0"
-               offset="0.0"/>
+        <limit lower="-0.02" upper="0.0" effort="100.0" velocity="0.5"/>
+        <mimic joint="left_finger_joint" multiplier="1.0" offset="0.0"/>
     </joint>
 </robot>

File: scara_description/urdf/gazebo.xacro (robot description, xacro)
@@ -1,23 +1,35 @@
 <?xml version="1.0"?>
 <robot xmlns:xacro="http://www.ros.org/wiki/xacro" name="scara">
-  <!-- ROS 2 Humble -->
-  <gazebo>
-    <xacro:if value="$(arg is_ignition)">
-      <plugin filename="ign_ros2_control-system" name="ign_ros2_control::IgnitionROS2ControlPlugin">
-        <parameters>$(find scara_controller)/config/scara_controllers.yaml</parameters>
-      </plugin>
-      <plugin filename="ignition-gazebo-sensors-system" name="ignition::gazebo::systems::Sensors">
-        <render_engine>ogre2</render_engine>
-      </plugin>
+    <!-- Declare args with defaults so xacro never errors if caller omits them -->
+    <xacro:arg name="is_sim"      default="true"/>
+    <xacro:arg name="is_ignition" default="false"/>
+    <xacro:if value="$(arg is_sim)">
+        <xacro:if value="$(arg is_ignition)">
+            <!-- ROS 2 Humble + Ignition Fortress -->
+            <gazebo>
+                <plugin filename="ign_ros2_control-system"
+                        name="ign_ros2_control::IgnitionROS2ControlPlugin">
+                    <parameters>$(find scara_controller)/config/scara_controllers.yaml</parameters>
+                </plugin>
+                <plugin filename="ignition-gazebo-sensors-system"
+                        name="ignition::gazebo::systems::Sensors">
+                    <render_engine>ogre2</render_engine>
+                </plugin>
+            </gazebo>
+        </xacro:if>
+        <xacro:unless value="$(arg is_ignition)">
+            <!-- ROS 2 Iron+ + Gazebo Garden/Harmonic -->
+            <gazebo>
+                <plugin filename="gz_ros2_control-system"
+                        name="gz_ros2_control::GazeboSimROS2ControlPlugin">
+                    <parameters>$(find scara_controller)/config/scara_controllers.yaml</parameters>
+                </plugin>
+                <plugin filename="gz-sim-sensors-system"
+                        name="gz::sim::systems::Sensors">
+                    <render_engine>ogre2</render_engine>
+                </plugin>
+            </gazebo>
+        </xacro:unless>
     </xacro:if>
-    <!-- ROS 2 Iron or above -->
-    <xacro:unless value="$(arg is_ignition)">
-      <plugin filename="gz_ros2_control-system" name="gz_ros2_control::GazeboSimROS2ControlPlugin">
-        <parameters>$(find scara_controller)/config/scara_controllers.yaml</parameters>
-      </plugin>
-      <plugin filename="gz-sim-sensors-system" name="gz::sim::systems::Sensors">
-        <render_engine>ogre2</render_engine>
-      </plugin>
-    </xacro:unless>
-  </gazebo>
+    <!-- No <gazebo> block needed when is_sim=false (display / slider GUI) -->
 </robot>

File: scara_description/urdf/scara.urdf.xacro (robot description, xacro)
@@ -4,4 +4,5 @@
     <xacro:arg name="is_sim" default="true"/>
     <xacro:include filename="$(find scara_description)/urdf/arm.xacro" />
+    <xacro:include filename="$(find scara_description)/urdf/materials.xacro" />
     <xacro:include filename="$(find scara_description)/urdf/gazebo.xacro" />
     <xacro:include filename="$(find scara_description)/urdf/ros2control.xacro" />
