Commit message: opencv gesture control added and urdf finger limits update

File: scara_description/urdf/arm.xacro (robot description, xacro)
@@ -191,5 +191,5 @@
         <child link="left_finger_link"/>
         <axis xyz="0 1 0"/>
-        <limit lower="-0.02" upper="0.0" effort="100.0" velocity="0.5"/>
+        <limit lower="-0.06" upper="0.0" effort="100.0" velocity="0.5"/>
     </joint>
     <!-- ── RIGHT FINGER ──────────────────────────────── -->
@@ -224,5 +224,5 @@
         <child link="right_finger_link"/>
         <axis xyz="0 -1 0"/>
-        <limit lower="-0.02" upper="0.0" effort="100.0" velocity="0.5"/>
+        <limit lower="-0.06" upper="0.0" effort="100.0" velocity="0.5"/>
         <mimic joint="left_finger_joint" multiplier="1.0" offset="0.0"/>
     </joint>

File: scara_description/urdf/ros2control.xacro (robot description, xacro)
@@ -64,5 +64,5 @@
         <joint name="left_finger_joint">
             <command_interface name="position">
-                <param name="min">-0.02</param>
+                <param name="min">-0.06</param>
                 <param name="max">0.0</param>
             </command_interface>

Commit message: moveit2 added, but controller fix required

File: scara_description/urdf/arm.xacro (robot description, xacro)
@@ -227,3 +227,9 @@
         <mimic joint="left_finger_joint" multiplier="1.0" offset="0.0"/>
     </joint>
+    <!-- DUMMY JOINT FOR MOVEIT2-->
+    <joint name="right_finger_joint_mimic" type="fixed">
+        <parent link="world"/>
+        <child link="right_finger_joint_mimic_dummy"/>
+    </joint>
+    <link name="right_finger_joint_mimic_dummy"/>
 </robot>

File: scara_description/urdf/materials.xacro (robot description, xacro)
@@ -1,7 +1,4 @@
 <?xml version="1.0"?>
 <robot xmlns:xacro="http://www.ros.org/wiki/xacro" name="scara">
-    <material name="scara_charcoal">
-        <color rgba="0.18 0.20 0.22 1.0"/>
-    </material>
     <material name="scara_dark_blue">
         <color rgba="0.08 0.28 0.55 1.0"/>
@@ -10,56 +7,6 @@
         <color rgba="0.12 0.45 0.80 1.0"/>
     </material>
-    <material name="scara_orange">
-        <color rgba="0.95 0.50 0.05 1.0"/>
-    </material>
     <material name="scara_light_grey">
         <color rgba="0.75 0.77 0.80 1.0"/>
     </material>
-    <!-- ═══════════════════════════════════════════════
-         GAZEBO MATERIALS  (<gazebo reference="...">)
-         Uses Gazebo built-in Gazebo/* material names
-         which map to Ogre materials with real shading.
-    ═══════════════════════════════════════════════ -->
-    <!-- base_link  — charcoal / near-black -->
-    <gazebo reference="base_link">
-        <material>Gazebo/Blue</material>
-        <mu1>0.9</mu1>
-        <mu2>0.9</mu2>
-    </gazebo>
-    <!-- column_link — dark navy blue -->
-    <gazebo reference="column_link">
-        <material>Gazebo/Blue</material>
-        <mu1>0.5</mu1>
-        <mu2>0.5</mu2>
-    </gazebo>
-    <!-- shoulder_link — mid blue -->
-    <gazebo reference="shoulder_link">
-        <material>Gazebo/SkyBlue</material>
-        <mu1>0.5</mu1>
-        <mu2>0.5</mu2>
-    </gazebo>
-    <!-- forearm_link — dark blue again (alternating) -->
-    <gazebo reference="forearm_link">
-        <material>Gazebo/SkyBlue</material>
-        <mu1>0.5</mu1>
-        <mu2>0.5</mu2>
-    </gazebo>
-    <!-- wrist_link — light grey accent -->
-    <gazebo reference="wrist_link">
-        <material>Gazebo/Grey</material>
-        <mu1>0.5</mu1>
-        <mu2>0.5</mu2>
-    </gazebo>
-    <!-- left_finger_link — orange gripper -->
-    <gazebo reference="left_finger_link">
-        <material>Gazebo/Orange</material>
-        <mu1>1.2</mu1>
-        <mu2>1.2</mu2>
-    </gazebo>
-    <!-- right_finger_link — orange gripper -->
-    <gazebo reference="right_finger_link">
-        <material>Gazebo/Orange</material>
-        <mu1>1.2</mu1>
-        <mu2>1.2</mu2>
-    </gazebo>
 </robot>

Commit message: world update & Pymoveit2

File: scara_description/urdf/arm.xacro (robot description, xacro)
@@ -94,5 +94,5 @@
         <child link="shoulder_link"/>
         <axis xyz="0 0 1"/>
-        <limit lower="-0.12" upper="0.02" effort="100.0" velocity="0.5"/>
+        <limit lower="-0.15" upper="0.02" effort="100.0" velocity="0.5"/>
     </joint>
     <!-- ── FOREARM ───────────────────────────────────── -->

Commit message: pymoveit2 added

File: scara_description/urdf/arm.xacro (robot description, xacro)
@@ -228,8 +228,8 @@
     </joint>
     <!-- DUMMY JOINT FOR MOVEIT2-->
+    <link name="right_finger_joint_mimic_dummy"/>
     <joint name="right_finger_joint_mimic" type="fixed">
         <parent link="world"/>
         <child link="right_finger_joint_mimic_dummy"/>
     </joint>
-    <link name="right_finger_joint_mimic_dummy"/>
 </robot>

Commit message: depth camera added , urdf

File: scara_description/urdf/arm.xacro (robot description, xacro)
@@ -94,5 +94,5 @@
         <child link="shoulder_link"/>
         <axis xyz="0 0 1"/>
-        <limit lower="-0.15" upper="0.02" effort="100.0" velocity="0.5"/>
+        <limit lower="-0.15" upper="0.02" effort="250.0" velocity="0.5"/>
     </joint>
     <!-- ── FOREARM ───────────────────────────────────── -->

File: scara_description/urdf/gazebo.xacro (robot description, xacro)
@@ -32,4 +32,52 @@
         </xacro:unless>
     </xacro:if>
-    <!-- No <gazebo> block needed when is_sim=false (display / slider GUI) -->
+    <!-- <gazebo reference="camera_link">
+        <sensor name="camera" type="camera">
+            <pose>0 0 0 0 0 0 </pose>
+            <visualize>true</visualize>
+            <update_rate>10.0</update_rate>
+            <alwaysOn>true</alwaysOn>
+            <topic>camera/image_raw</topic>
+            <gz_frame_id>camera_link_optical</gz_frame_id>
+            <camera name="intel_realsense_r200">
+                <camera_info_topic>camera/camera_info</camera_info_topic>
+                <horizontal_fov>1.3962634</horizontal_fov>
+                <image>
+                    <width>640</width>
+                    <height>480</height>
+                    <format>R8G8B8</format>
+                </image>
+                <clip>
+                    <near>0.05</near>
+                    <far>8.0</far>
+                </clip>
+            </camera>
+        </sensor>
+    </gazebo> -->
+    <gazebo reference="camera_link">
+    <sensor name="camera" type="camera">
+        <pose>0 0 0 0 0 0</pose>
+        <visualize>true</visualize>
+        <update_rate>10.0</update_rate>
+        <alwaysOn>true</alwaysOn>
+        <topic>camera/image_raw</topic>
+        <gz_frame_id>camera_link_optical</gz_frame_id>
+        <camera name="intel_realsense_r200">
+        <camera_info_topic>camera/camera_info</camera_info_topic>
+        <horizontal_fov>1.3962634</horizontal_fov>
+        <image>
+            <width>640</width>
+            <height>480</height>
+            <format>R8G8B8</format>
+        </image>
+        <clip>
+            <near>0.05</near>
+            <far>8.0</far>
+        </clip>
+        <depth_camera>
+            <output>depths</output>
+        </depth_camera>
+        </camera>
+    </sensor>
+    </gazebo>
 </robot>

File: scara_description/urdf/scara.urdf.xacro (robot description, xacro)
@@ -4,4 +4,5 @@
     <xacro:arg name="is_sim" default="true"/>
     <xacro:include filename="$(find scara_description)/urdf/arm.xacro" />
+    <xacro:include filename="$(find scara_description)/urdf/camera.xacro" />
     <xacro:include filename="$(find scara_description)/urdf/materials.xacro" />
     <xacro:include filename="$(find scara_description)/urdf/gazebo.xacro" />

Commit message: vision pnp added

File: scara_description/urdf/arm.xacro (robot description, xacro)
@@ -159,4 +159,11 @@
         <axis xyz="0 0 1"/>
         <limit lower="-2.0" upper="2.0" effort="10.0" velocity="1.5"/>
+    </joint>
+    <!-- Tool centre point: centre of the gripper finger tips. -->
+    <link name="tool0"/>
+    <joint name="tool0_joint" type="fixed">
+        <parent link="wrist_link"/>
+        <child link="tool0"/>
+        <origin xyz="0.08 0 -0.10" rpy="0 0 0"/>
     </joint>
     <!-- ── LEFT FINGER ───────────────────────────────── -->
